File: Footprint Test/SparkFun_SMD_LED_Light_Pipe_Footprint_Test.kicad_pcb (KiCad board)
At the start: 2 copper layers, 21.3 x 33 mm, 21 parts, among them J1 Conn_01x04

Commit message: Update footprint name
Parts:
- REF** (x2): footprint SparkFun SMD LED Light Pipe:SMD-CBI-5mm -> SparkFun SMD LED Light Pipe:SparkFun_SMD_LED_Light_Pipe-5mm
- REF**: footprint SparkFun SMD LED Light Pipe:SMD-CBI-5mm-4Gang -> SparkFun SMD LED Light Pipe:SparkFun_SMD_LED_Light_Pipe-5mm-4Gang
Changed lines of the file:
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@@
 		)
 	)
-	(footprint "SparkFun SMD LED Light Pipe:SMD-CBI-5mm"
+	(footprint "SparkFun SMD LED Light Pipe:SparkFun_SMD_LED_Light_Pipe-5mm"
 		(layer "F.Cu")
 		(at 97.155 79.375 -90)
-		(tags "SparkFun SMD 5mm Light Pipe Circuit Board Indicator")
+		(tags "SparkFun SMD LED 5mm Light Pipe Circuit Board Indicator CBI")
 		(property "Reference" "REF**"
 			(at 0 -4.7 -90)
@@
 			)
 		)
-		(property "Footprint" "SparkFun SMD LED Light Pipe:SMD-CBI-5mm"
+		(property "Footprint" "SparkFun SMD LED Light Pipe:SparkFun_SMD_LED_Light_Pipe-5mm"
 			(at 0 -4.800001 -90)
 			(unlocked yes)
@@
 		)
 		(property "Datasheet" ""
-			(at 0 0 -90)
+			(at 0 5.715 -90)
 			(unlocked yes)
 			(layer "F.Fab")
@@
 			(effects
 				(font
-					(size 1 1)
-					(thickness 0.15)
+					(size 0.5 0.5)
+					(thickness 0.1)
 				)
 			)
@@
 		)
 		(fp_rect
-			(start -3.429 2.667)
+			(start -1.905 2.413)
 			(end 1.905 4.064)
 			(stroke
@@
 		)
 		(fp_rect
-			(start -3.429 -2.54)
-			(end -2.032 2.54)
+			(start -3.429 -4.064)
+			(end -2.032 4.064)
 			(stroke
 				(width 0.05)
@@
 		)
 		(fp_rect
-			(start -3.429 -4.064)
-			(end 1.905 -2.667)
+			(start -1.905 -4.064)
+			(end 1.905 -2.413)
 			(stroke
 				(width 0.05)
@@
 		)
 	)
-	(footprint "SparkFun SMD LED Light Pipe:SMD-CBI-5mm"
+	(footprint "SparkFun SMD LED Light Pipe:SparkFun_SMD_LED_Light_Pipe-5mm"
 		(layer "F.Cu")
 		(at 97.155 55.245 90)
-		(tags "SparkFun SMD 5mm Light Pipe Circuit Board Indicator")
+		(tags "SparkFun SMD LED 5mm Light Pipe Circuit Board Indicator CBI")
 		(property "Reference" "REF**"
 			(at 0 -4.7 90)
@@
 			)
 		)
-		(property "Footprint" "SparkFun SMD LED Light Pipe:SMD-CBI-5mm"
+		(property "Footprint" "SparkFun SMD LED Light Pipe:SparkFun_SMD_LED_Light_Pipe-5mm"
 			(at 0 -4.800001 90)
 			(unlocked yes)
@@
 		)
 		(property "Datasheet" ""
-			(at 0 0 90)
+			(at 0 5.715 90)
 			(unlocked yes)
 			(layer "F.Fab")
@@
 			(effects
 				(font
-					(size 1 1)
-					(thickness 0.15)
+					(size 0.5 0.5)
+					(thickness 0.1)
 				)
 			)
@@
 		)
 		(fp_rect
-			(start -3.429 -4.064)
-			(end 1.905 -2.667)
+			(start -1.905 -4.064)
+			(end 1.905 -2.413)
 			(stroke
 				(width 0.05)
@@
 		)
 		(fp_rect
-			(start -3.429 -2.54)
-			(end -2.032 2.54)
+			(start -3.429 -4.064)
+			(end -2.032 4.064)
 			(stroke
 				(width 0.05)
@@
 		)
 		(fp_rect
-			(start -3.429 2.667)
+			(start -1.905 2.413)
 			(end 1.905 4.064)
 			(stroke
@@
 		)
 		(group ""
-			(members "194f3fdf-8d05-4a50-97a1-5c5e2c99950f" "2470e73c-90c9-4dad-a487-9f423d5fae9c"
-				"3dd6a5dd-9faf-4fa9-9c08-b4f71db8bc7d" "59b944e4-855f-4b3c-b418-89a38fae9e61"
-				"8a2b91ea-5536-4fd2-959f-ab6984814f90" "9e972bd6-114b-4d3d-8485-f60deff10494"
-				"a1a556bf-c5eb-48b9-a919-c450ee973301" "a7ea713c-b795-4aad-b297-57c1cac86a5f"
-				"b5ef2b28-c866-4bbb-b553-9a0c2f4daac3"
+			(members "2b5cc1a9-eeef-4695-be68-b520b8dc1586" "4ddb896e-3397-4b20-b00f-0a9418a33848"
+				"6227c80e-8721-4195-a372-a23ed5bac137" "6ef9e509-f150-4be4-a574-eccc6061afd5"
+				"928002d3-5d86-4919-a1ad-3c2fc18d5fe7" "9cc44372-57c5-47de-bd8a-a4b4213e0bb6"
+				"a4487fde-d98e-44f3-94a7-c134fd46174c" "c65c16f4-9f90-4c32-9750-0d70904e12b9"
+				"d502631d-ff7c-4c29-b9e0-b0a58c097781"
 			)
 		)
@@
 		)
 	)
-	(footprint "SparkFun SMD LED Light Pipe:SMD-CBI-5mm-4Gang"
+	(footprint "SparkFun SMD LED Light Pipe:SparkFun_SMD_LED_Light_Pipe-5mm-4Gang"
 		(layer "F.Cu")
 		(at 108.9025 78.675)
+		(tags "SparkFun SMD LED 5mm Light Pipe Circuit Board Indicator CBI")
 		(property "Reference" "REF**"
 			(at 0 -27.305 0)
@@
 			)
 		)
-		(property "Footprint" "SparkFun SMD LED Light Pipe:SMD-CBI-5mm-4Gang"
+		(property "Footprint" "SparkFun SMD LED Light Pipe:SparkFun_SMD_LED_Light_Pipe-5mm-4Gang"
 			(at 0.6 -28.125 0)
 			(unlocked yes)
@@
 		)
 		(property "Datasheet" ""
-			(at 0 0 0)
+			(at 0 6.096 0)
 			(unlocked yes)
 			(layer "F.Fab")
@@
 			(effects
 				(font
-					(size 1 1)
-					(thickness 0.15)
+					(size 0.5 0.5)
+					(thickness 0.1)
 				)
 			)
