File: Footprint Test/SparkFun_SMD_LED_Light_Pipe_Footprint_Test.kicad_sch (KiCad schematic)
At the start: 10 parts, among them J1 Conn_01x04

Commit message: Update layout with 3D model
Parts:
- D2: footprint SparkFun-LED:LED_0603_1608Metric -> SparkFun-LED:LED_0603_1608Metric_Blue
Changed lines of the file:
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@@
 			)
 		)
-		(property "Footprint" "SparkFun-LED:LED_0603_1608Metric"
+		(property "Footprint" "SparkFun-LED:LED_0603_1608Metric_Blue"
 			(at 38.1 59.69 0)
 			(effects
